Commit message: added launch files

File: src/igvc_test_description/robot.urdf (robot description, URDF)
Before this commit: robot igvc_bot2, 6 links, 5 joints
Links:
- link caster_raceway_link: geometry collision mesh filename=package://igvc_test_description/meshes/Part_2.obj scale=1. 1. 1.; visual mesh filename=package://igvc_test_description/meshes/Part_2.obj scale=1. 1. 1.
- link caster_wheel_link: geometry collision mesh filename=package://igvc_test_description/meshes/_in_Caster.obj scale=1. 1. 1.; visual mesh filename=package://igvc_test_description/meshes/_in_Caster.obj scale=1. 1. 1.
- link chassis_link: geometry collision mesh filename=package://igvc_test_description/meshes/_FE2CBA3_2B86_49A6_8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 scale=1. 1. 1.; visual mesh filename=package://igvc_test_description/meshes/_FE2CBA3_2B86_49A6_8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 scale=1. 1. 1.
- link left_wheel_link: geometry collision mesh filename=package://igvc_test_description/meshes/left_wheel_link__in_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 scale=1. 1. 1.; visual mesh filename=package://igvc_test_description/meshes/left_wheel_link__in_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 scale=1. 1. 1.
- link right_wheel_link: geometry collision mesh filename=package://igvc_test_description/meshes/right_wheel_link__in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 scale=1. 1. 1.; visual mesh filename=package://igvc_test_description/meshes/right_wheel_link__in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 scale=1. 1. 1.

File: src/igvc_test_description/urdf/control/ros2_control_info.urdf.xacro (robot description, xacro)
@@ -1,4 +1,5 @@
 <?xml version="1.0"?>
 <robot xmlns:xacro="http://www.ros.org/wiki/xacro">
+  <xacro:arg name="hardware_interface" default="IsaacDriveHardware" />
   <ros2_control name="igvc_test_bot" type="system">
     <hardware>
