Commit message: temp changes to urdf

File: src/igvc_test_description/robot2.urdf (robot description, URDF)
Before this commit: robot igvc_test_robot, 27 links, 26 joints
Links:
- link front_zed_camera_x_camera_center: geometry collision mesh filename=file:///workspace/DevEnv/jazzy_ws/IGVC_robot_2026/jazzy_ws/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; visual mesh filename=file:///workspace/DevEnv/jazzy_ws/IGVC_robot_2026/jazzy_ws/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
- link left_zed_camera_x_camera_center: geometry collision mesh filename=file:///workspace/DevEnv/jazzy_ws/IGVC_robot_2026/jazzy_ws/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; visual mesh filename=file:///workspace/DevEnv/jazzy_ws/IGVC_robot_2026/jazzy_ws/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
- link right_zed_camera_x_camera_center: geometry collision mesh filename=file:///workspace/DevEnv/jazzy_ws/IGVC_robot_2026/jazzy_ws/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; visual mesh filename=file:///workspace/DevEnv/jazzy_ws/IGVC_robot_2026/jazzy_ws/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

Commit message: updated urdf

File: src/igvc_test_description/robot2.urdf (robot description, URDF)
Before this commit: robot igvc_test_robot, 27 links, 26 joints
Links:
- link front_zed_camera_x_camera_center: geometry collision mesh filename=file:///workspace/DevEnv/jazzy_ws/IGVC_robot_2026/install/z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; visual mesh filename=file:///workspace/DevEnv/jazzy_ws/IGVC_robot_2026/install/z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
- link left_zed_camera_x_camera_center: geometry collision mesh filename=file:///workspace/DevEnv/jazzy_ws/IGVC_robot_2026/install/z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; visual mesh filename=file:///workspace/DevEnv/jazzy_ws/IGVC_robot_2026/install/z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
- link right_zed_camera_x_camera_center: geometry collision mesh filename=file:///workspace/DevEnv/jazzy_ws/IGVC_robot_2026/install/z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; visual mesh filename=file:///workspace/DevEnv/jazzy_ws/IGVC_robot_2026/install/z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
