Commit message: updated urdf

File: src/igvc_test_description/urdf/control/ros2_control_info.urdf.xacro (robot description, xacro)
@@ -4,4 +4,9 @@
   <ros2_control name="igvc_test_bot" type="system">
     <hardware>
+      <param name="can_interface">can0</param>
+      <param name="joint_map">right_wheel_joint:R, left_wheel_joint:L</param>
+      <param name="can_id_map"><R:0x100:0x101,L:0x100:0x101></param>
+      <param name="invert_can_joints">R</param>
+      <param name="controlled_joints">right_wheel_joint, left_wheel_joint</param>
       <plugin>grr_hardware/$(arg hardware_interface)</plugin>
     </hardware>

File: src/igvc_test_description/urdf/parts/test_robot_body.urdf.xacro (robot description, xacro)
@@ -2,137 +2,129 @@
 <robot xmlns:xacro="http://www.ros.org/wiki/xacro">
     <xacro:macro name="robot_body">
-        <joint name="right_wheel_joint" type="continuous">
-            <origin xyz="-0.25135 0. -0.128425" rpy="-1.5707966 -0.0000001 -1.5707964" />
-            <parent link="chassis_link" />
-            <child link="right_wheel_link" />
-            <axis xyz="0. 0. 1." />
-        </joint>
-        <joint name="caster_raceway_joint" type="continuous">
-            <origin xyz="0. -0.3725 -0.044525" rpy="3.1415927 0. 0. " />
-            <parent link="chassis_link" />
-            <child link="caster_raceway_link" />
-            <axis xyz="0. 0. 1." />
-        </joint>
-        <joint name="left_wheel_joint" type="continuous">
-            <origin xyz="0.25135 0. -0.128425" rpy="3.1415927 1.5707964 0. " />
-            <parent link="chassis_link" />
-            <child link="left_wheel_link" />
-            <axis xyz="0. 0. -1." />
-        </joint>
-        <joint name="caster_wheel_joint" type="continuous">
-            <origin xyz="-0.0270522 -0.0350281 0.1085062" rpy="1.5707963 0.0862497 -1.660313 " />
-            <parent link="caster_raceway_link" />
-            <child link="caster_wheel_link" />
-            <axis xyz="0. 0. -1." />
-        </joint>
-        <joint name="rootJoint" type="fixed">
-            <origin xyz="0. 0. 0." rpy="0. 0. 0." />
-            <parent link="base_link" />
-            <child link="chassis_link" />
-        </joint>
-        <link name="caster_raceway_link">
-            <visual>
-                <origin xyz="0. -0. -0.005" rpy="-3.1415927 0. 1.4812796" />
-                <geometry>
-                    <mesh filename="package://igvc_test_description/meshes/Part_2.obj"
-                        scale="1. 1. 1." />
-                </geometry>
-            </visual>
-            <collision>
-                <origin xyz="0. -0. -0.005" rpy="-3.1415927 0. 1.4812796" />
-                <geometry>
-                    <mesh filename="package://igvc_test_description/meshes/Part_2.obj"
-                        scale="1. 1. 1." />
-                </geometry>
-            </collision>
-        </link>
-        <link name="caster_wheel_link">
-            <inertial>
-                <origin xyz="0. 0. -0.0238125" rpy="0. 0. 0." />
-                <mass value="1.0005643" />
-                <inertia ixx="0.0017247" ixy="-0." ixz="-0." iyy="0.0030953" iyz="0."
-                    izz="0.0017247" />
-            </inertial>
-            <visual>
-                <origin xyz="0.0373062 0.1135063 -0.0238125" rpy="-1.5707963 -0. 0.0000001" />
-                <geometry>
-                    <mesh filename="package://igvc_test_description/meshes/_in_Caster.obj"
-                        scale="1. 1. 1." />
-                </geometry>
-            </visual>
-            <collision>
-                <origin xyz="0.0373062 0.1135063 -0.0238125" rpy="-1.5707963 -0. 0.0000001" />
-                <geometry>
-                    <mesh filename="package://igvc_test_description/meshes/_in_Caster.obj"
-                        scale="1. 1. 1." />
-                </geometry>
-            </collision>
-        </link>
-        <link name="chassis_link">
-            <visual>
-                <origin xyz="0. 0. 0." rpy="0. 0. 0." />
-                <geometry>
-                    <mesh
-                        filename="package://igvc_test_description/meshes/_FE2CBA3_2B86_49A6_86C6_46C335366A6A.obj"
-                        scale="1. 1. 1." />
-                </geometry>
-            </visual>
-            <collision>
-                <origin xyz="0. 0. 0." rpy="0. 0. 0." />
-                <geometry>
-                    <mesh
-                        filename="package://igvc_test_description/meshes/_FE2CBA3_2B86_49A6_86C6_46C335366A6A.obj"
-                        scale="1. 1. 1." />
-                </geometry>
-            </collision>
-        </link>
-        <link name="base_link" />
-        <link name="left_wheel_link">
-            <inertial>
-                <origin xyz="0. 0. -0.032" rpy="0. 0. 0." />
-                <mass value="2.1118586" />
-                <inertia ixx="0.0059185" ixy="0." ixz="0." iyy="0.0105056" iyz="-0." izz="0.0059185" />
-            </inertial>
-            <visual>
-                <origin xyz="0. 0. -0.032" rpy="1.5707964 0. 0. " />
-                <geometry>
-                    <mesh
-                        filename="package://igvc_test_description/meshes/left_wheel_link__in_Wheel_Stand_In.obj"
-                        scale="1. 1. 1." />
-                </geometry>
-            </visual>
-            <collision>
-                <origin xyz="0. 0. -0.032" rpy="1.5707964 0. 0. " />
-                <geometry>
-                    <mesh
-                        filename="package://igvc_test_description/meshes/left_wheel_link__in_Wheel_Stand_In.obj"
-                        scale="1. 1. 1." />
-                </geometry>
-            </collision>
-        </link>
-        <link name="right_wheel_link">
-            <inertial>
-                <origin xyz="0. 0. -0.032" rpy="0. 0. 0." />
-                <mass value="2.1118586" />
-                <inertia ixx="0.0059185" ixy="-0." ixz="-0." iyy="0.0105056" iyz="0."
-                    izz="0.0059185" />
-            </inertial>
-            <visual>
-                <origin xyz="0. 0. -0.032" rpy="-1.5707961 -0.0000001 0.0000001" />
-                <geometry>
-                    <mesh
-                        filename="package://igvc_test_description/meshes/right_wheel_link__in_Wheel_Stand_In.obj"
-                        scale="1. 1. 1." />
-                </geometry>
-            </visual>
-            <collision>
-                <origin xyz="0. 0. -0.032" rpy="-1.5707961 -0.0000001 0.0000001" />
-                <geometry>
-                    <mesh
-                        filename="package://igvc_test_description/meshes/right_wheel_link__in_Wheel_Stand_In.obj"
-                        scale="1. 1. 1." />
-                </geometry>
-            </collision>
-        </link>
+  <joint name="caster_raceway_joint" type="continuous">
+    <origin xyz="0.0011449 -0.3728886 -0.0307033" rpy="0. 0. 0."/>
+    <parent link="temp"/>
+    <child link="caster_raceway_link"/>
+    <axis xyz="0. 0. 1."/>
+  </joint>
+  <joint name="caster_wheel_joint" type="continuous">
+    <origin xyz="-0.0452015 0.004609 -0.1223279" rpy="-1.5707961 -0.0862496 2.4779847"/>
+    <parent link="caster_raceway_link"/>
+    <child link="caster_wheel_link"/>
+    <axis xyz="0. 0. 1."/>
+  </joint>
+  <joint name="left_wheel_joint" type="continuous">
+    <origin xyz="0.2844359 0.1500906 -0.1274171" rpy="0. 0. 0."/>
+    <parent link="temp"/>
+    <child link="left_wheel_link"/>
+    <axis xyz="1. 0. 0."/>
+  </joint>
+  <joint name="right_wheel_joint" type="continuous">
+    <origin xyz="-0.2918941 0.1492591 -0.1296445" rpy="0. 0. 0."/>
+    <parent link="temp"/>
+    <child link="right_wheel_link"/>
+    <axis xyz="1. 0. 0."/>
+  </joint>
+  <joint name="rootJoint" type="fixed">
+    <origin xyz="0. 0. 0." rpy="0. 0. -0."/>
+    <parent link="temp"/>
+    <child link="base_link"/>
+  </joint>
+  <link name="base_link"/>
+  <link name="caster_raceway_link">
+    <inertial>
+      <origin xyz="-0.0118137 0.0087306 -0.0584325" rpy="0. 0. 0."/>
+      <mass value="0.2597675"/>
+      <inertia ixx="0.0003673" ixy="0.0001647" ixz="0." iyy="0.0004492" iyz="-0." izz="0.0006678"/>
+    </inertial>
+    <visual>
+      <origin xyz="-0.0011449 0.0003886 -0.0088217" rpy="0. 0. -0.663608"/>
+      <geometry>
+        <mesh filename="package://igvc_test_description/meshes/caster_raceway_link_Part_2_Part_2.obj" scale="1. 1. 1."/>
+      </geometry>
+    </visual>
+    <collision>
+      <origin xyz="-0.0011449 0.0003886 -0.0088217" rpy="0. 0. -0.663608"/>
+      <geometry>
+        <mesh filename="package://igvc_test_description/meshes/caster_raceway_link_Part_2_Part_2.obj" scale="1. 1. 1."/>
+      </geometry>
+    </collision>
+  </link>
+  <link name="caster_wheel_link">
+    <inertial>
+      <origin xyz="-0. -0. -0.0238125" rpy="0. 0. 0."/>
+      <mass value="1.0005643"/>
+      <inertia ixx="0.0017247" ixy="-0." ixz="0." iyy="0.0030953" iyz="-0." izz="0.0017247"/>
+    </inertial>
+    <visual>
+      <origin xyz="0.0373062 0.1135063 -0.0238125" rpy="-1.5707965 -0.0000001 0. "/>
+      <geometry>
+        <mesh filename="package://igvc_test_description/meshes/caster_wheel_link__in_Caster__in_Caster.obj" scale="1. 1. 1."/>
+      </geometry>
+    </visual>
+    <collision>
+      <origin xyz="0.0373062 0.1135063 -0.0238125" rpy="-1.5707965 -0.0000001 0. "/>
+      <geometry>
+        <mesh filename="package://igvc_test_description/meshes/caster_wheel_link__in_Caster__in_Caster.obj" scale="1. 1. 1."/>
+      </geometry>
+    </collision>
+  </link>
+  <link name="left_wheel_link">
+    <inertial>
+      <origin xyz="-0.0010859 -0.0000906 -0.0010079" rpy="0. 0. 0."/>
+      <mass value="2.1118586"/>
+      <inertia ixx="0.0059185" ixy="-0." ixz="-0." iyy="0.0086441" iyz="0.0022525" izz="0.00778"/>
+    </inertial>
+    <visual>
+      <origin xyz="-0.0010859 -0.0000906 -0.0010079" rpy="0. 0.8801533 1.5707964"/>
+      <geometry>
+        <mesh filename="package://igvc_test_description/meshes/left_wheel_link__in_Wheel_Stand_In_01__in_Wheel_Stand_In.obj" scale="1. 1. 1."/>
+      </geometry>
+    </visual>
+    <collision>
+      <origin xyz="-0.0010859 -0.0000906 -0.0010079" rpy="0. 0.8801533 1.5707964"/>
+      <geometry>
+        <mesh filename="package://igvc_test_description/meshes/left_wheel_link__in_Wheel_Stand_In_01__in_Wheel_Stand_In.obj" scale="1. 1. 1."/>
+      </geometry>
+    </collision>
+  </link>
+  <link name="right_wheel_link">
+    <inertial>
+      <origin xyz="0.0085441 0.0007409 0.0012195" rpy="0. 0. 0."/>
+      <mass value="2.1118586"/>
+      <inertia ixx="0.0059185" ixy="-0." ixz="0." iyy="0.0059185" iyz="-0." izz="0.0105056"/>
+    </inertial>
+    <visual>
+      <origin xyz="0.0085441 0.0007409 0.0012195" rpy="3.1415927 0. -1.5707964"/>
+      <geometry>
+        <mesh filename="package://igvc_test_description/meshes/right_wheel_link__in_Wheel_Stand_In_01__in_Wheel_Stand_In.obj" scale="1. 1. 1."/>
+      </geometry>
+    </visual>
+    <collision>
+      <origin xyz="0.0085441 0.0007409 0.0012195" rpy="3.1415927 0. -1.5707964"/>
+      <geometry>
+        <mesh filename="package://igvc_test_description/meshes/right_wheel_link__in_Wheel_Stand_In_01__in_Wheel_Stand_In.obj" scale="1. 1. 1."/>
+      </geometry>
+    </collision>
+  </link>
+  <link name="temp">
+    <inertial>
+      <origin xyz="0. 0. 0." rpy="0. 0. 0."/>
+      <mass value="20."/>
+      <inertia ixx="0.001" ixy="0." ixz="0." iyy="0.001" iyz="0." izz="0.001"/>
+    </inertial>
+    <visual>
+      <origin xyz="0. 0. 0." rpy="0. 0. 0."/>
+      <geometry>
+        <mesh filename="package://igvc_test_description/meshes/_FE2CBA3_2B86_49A6_86C6_46C335366A6A.obj" scale="1. 1. 1."/>
+      </geometry>
+    </visual>
+    <collision>
+      <origin xyz="0. 0. 0." rpy="0. 0. 0."/>
+      <geometry>
+        <mesh filename="package://igvc_test_description/meshes/_FE2CBA3_2B86_49A6_86C6_46C335366A6A.obj" scale="1. 1. 1."/>
+      </geometry>
+    </collision>
+  </link>
     </xacro:macro>
 </robot>

File: src/igvc_test_description/urdf/robots/test_robot.urdf.xacro (robot description, xacro)
@@ -7,11 +7,11 @@
     <xacro:robot_body />
     <xacro:zed_camera_x parent="chassis_link" prefix="left">
-        <origin xyz="0.2 -0.1 0" rpy="0 0 ${3.14/3}"/>
+        <origin xyz="0.2 -0.1 ${3.14/2}" rpy="0 0 0"/>
     </xacro:zed_camera_x>
     <xacro:zed_camera_x parent="chassis_link" prefix="front">
-        <origin xyz="0.2 0.1 0" rpy="0 0 0"/>
+        <origin xyz="0.2 0 0" rpy="0 0 0"/>
     </xacro:zed_camera_x>
     <xacro:zed_camera_x parent="chassis_link" prefix="right">
-        <origin xyz="0.2 0.1 0" rpy="0 0 -${3.14/3}"/>
+        <origin xyz="0.2 0.1 -${3.14/2}" rpy="0 0 0"/>
     </xacro:zed_camera_x>
 </robot>

Commit message: syntax error

File: src/igvc_test_description/urdf/control/ros2_control_info.urdf.xacro (robot description, xacro)
@@ -2,8 +2,9 @@
 <robot xmlns:xacro="http://www.ros.org/wiki/xacro">
   <xacro:arg name="hardware_interface" default="IsaacDriveHardware" />
+  <xacro:property name="hardware_interface_value" value="$(arg hardware_interface)" />
   <ros2_control name="igvc_test_bot" type="system">
     <hardware>
       <plugin>grr_hardware/$(arg hardware_interface)</plugin>
-      <xacro:if value="${'$(arg hardware_interface)' == 'CanInterface'}">
+      <xacro:if value="${hardware_interface_value == 'CanInterface'}">
         <param name="can_interface">can0</param>
         <param name="joint_map">right_wheel_joint:R, left_wheel_joint:L</param>
