Commit message: working simulation interface

File: src/igvc_test_description/urdf/robots/test_robot.urdf.xacro (robot description, xacro)
@@ -3,5 +3,15 @@
     <xacro:include filename="$(find igvc_test_description)/urdf/parts/test_robot_body.urdf.xacro" />
     <xacro:include filename="$(find igvc_test_description)/urdf/control/ros2_control_info.urdf.xacro" />
+    <xacro:include filename="$(find igvc_test_description)/urdf/parts/zed_camera_x.urdf.xacro" />
     <xacro:arg name="hardware_interface" default="IsaacDriveHardware" />
     <xacro:robot_body />
+    <xacro:zed_camera_x parent="chassis_link" prefix="left">
+        <origin xyz="0.2 -0.1 ${3.14/2}" rpy="0 0 0"/>
+    </xacro:zed_camera_x>
+    <xacro:zed_camera_x parent="chassis_link" prefix="front">
+        <origin xyz="0.2 0 0" rpy="0 0 0"/>
+    </xacro:zed_camera_x>
+    <xacro:zed_camera_x parent="chassis_link" prefix="right">
+        <origin xyz="0.2 0.1 -${3.14/2}" rpy="0 0 0"/>
+    </xacro:zed_camera_x>
 </robot>

Commit message: temp changes to urdf

File: src/igvc_test_description/urdf/robots/test_robot.urdf.xacro (robot description, xacro)
@@ -7,11 +7,11 @@
     <xacro:robot_body />
     <xacro:zed_camera_x parent="chassis_link" prefix="left">
-        <origin xyz="0.2 -0.1 ${3.14/2}" rpy="0 0 0"/>
+        <origin xyz="0.2 -0.1 0" rpy="0 0 ${3.14/3}"/>
     </xacro:zed_camera_x>
     <xacro:zed_camera_x parent="chassis_link" prefix="front">
-        <origin xyz="0.2 0 0" rpy="0 0 0"/>
+        <origin xyz="0.2 0.1 0" rpy="0 0 0"/>
     </xacro:zed_camera_x>
     <xacro:zed_camera_x parent="chassis_link" prefix="right">
-        <origin xyz="0.2 0.1 -${3.14/2}" rpy="0 0 0"/>
+        <origin xyz="0.2 0.1 0" rpy="0 0 -${3.14/3}"/>
     </xacro:zed_camera_x>
 </robot>

Commit message: urdf updates

File: src/igvc_test_description/urdf/robots/test_robot.urdf.xacro (robot description, xacro)
@@ -9,11 +9,11 @@
     <xacro:robot_body />
     <xacro:zed_camera_x parent="chassis_link" prefix="left">
-        <origin xyz="0.4 0.2 0.194" rpy="0 ${3.14/18} ${3.14*95/180}"/>
+        <origin xyz="0.361 0.18 0.248" rpy="0 ${3.14/18} ${3.14*95/180}"/>
     </xacro:zed_camera_x>
     <xacro:zed_camera_x parent="chassis_link" prefix="front">
-        <origin xyz="0.45 0 0.194" rpy="0 0 0"/>
+        <origin xyz="0.405 0 0.246" rpy="0 0 0"/>
     </xacro:zed_camera_x>
     <xacro:zed_camera_x parent="chassis_link" prefix="right">
-        <origin xyz="0.4 -0.2 0.194" rpy="0 ${3.14/18} -${3.14*95/180}"/>
+        <origin xyz="0.359 -0.195 0.251" rpy="0 ${3.14/18} -${3.14*95/180}"/>
     </xacro:zed_camera_x>
     <xacro:rplidar_c1 parent="chassis_link" prefix="top">
@@ -21,5 +21,5 @@
     </xacro:rplidar_c1>
     <xacro:gps_antenna parent="chassis_link" prefix="front">
-        <origin xyz="0.2 -0.15 0.16" rpy="0 0 0"/>
+        <origin xyz="0.177 -0.133 0.218" rpy="0 0 0"/>
     </xacro:gps_antenna>
 </robot>

Commit message: tensorrt changes

File: src/igvc_test_description/urdf/robots/test_robot.urdf.xacro (robot description, xacro)
@@ -9,5 +9,5 @@
     <xacro:robot_body />
     <xacro:zed_camera_x parent="chassis_link" prefix="left">
-        <origin xyz="0.361 0.18 0.248" rpy="0 ${3.14/18} ${3.14*95/180}"/>
+        <origin xyz="0.361 0.18 0.248" rpy="0 ${3.14/18} ${3.14/4}"/>
     </xacro:zed_camera_x>
     <xacro:zed_camera_x parent="chassis_link" prefix="front">
@@ -15,5 +15,5 @@
     </xacro:zed_camera_x>
     <xacro:zed_camera_x parent="chassis_link" prefix="right">
-        <origin xyz="0.359 -0.195 0.251" rpy="0 ${3.14/18} -${3.14*95/180}"/>
+        <origin xyz="0.359 -0.195 0.251" rpy="0 ${3.14/18} -${3.14/4}"/>
     </xacro:zed_camera_x>
     <xacro:rplidar_c1 parent="chassis_link" prefix="top">

Commit message: added zed camera

File: src/igvc_test_description/urdf/robots/test_robot.urdf.xacro (robot description, xacro)
@@ -6,4 +6,5 @@
     <xacro:include filename="$(find igvc_test_description)/urdf/parts/rplidar_c1.urdf.xacro" />
     <xacro:include filename="$(find igvc_test_description)/urdf/parts/gps_antenna.urdf.xacro" />
+    <xacro:include filename="$(find igvc_test_description)/urdf/parts/zed_camera_2i.urdf.xacro" />
     <xacro:arg name="hardware_interface" default="IsaacDriveHardware" />
     <xacro:robot_body />
@@ -17,4 +18,7 @@
         <origin xyz="0.359 -0.195 0.251" rpy="0 ${3.14/18} -${3.14/4}"/>
     </xacro:zed_camera_x>
+    <xacro:zed_camera_2i parent="chassis_link" prefix="front">
+        <origin xyz="-0.215 0 0.248" rpy="0  0 0"/>
+    </xacro:zed_camera_2i>
     <xacro:rplidar_c1 parent="chassis_link" prefix="top">
         <origin xyz="0.225 0 0.46" rpy="0 0 0"/>
