Commit message: explosive changes

File: src/igvc_test_description/urdf/parts/zed_camera_x.urdf.xacro (robot description, xacro)
@@ -2,4 +2,14 @@
 <robot xmlns:xacro="http://www.ros.org/wiki/xacro">
 <xacro:include filename="$(find zed_description)/urdf/zed_macro.urdf.xacro"/>
+    <xacro:macro name="zed_camera_2i" params="parent *origin prefix">
+        <xacro:zed_camera name="${prefix}_zed_camera_2i" model="zed2i" enable_gnss="true">
+            <gnss_origin xyz="0 0 0" rpy="0 0 0"/>
+        </xacro:zed_camera>
+        <joint name="${prefix}_zed_camera_x_joint" type="fixed">
+            <parent link="${parent}"/>
+            <child link="${prefix}_zed_camera_x_camera_link"/>
+            <xacro:insert_block name="origin"/>
+        </joint>
+    </xacro:macro>
     <xacro:macro name="zed_camera_x" params="parent *origin prefix">
         <xacro:zed_camera name="${prefix}_zed_camera_x" model="zedx" enable_gnss="true">

File: src/igvc_test_description/urdf/robots/test_robot.urdf.xacro (robot description, xacro)
@@ -6,5 +6,5 @@
     <xacro:include filename="$(find igvc_test_description)/urdf/parts/rplidar_c1.urdf.xacro" />
     <xacro:include filename="$(find igvc_test_description)/urdf/parts/gps_antenna.urdf.xacro" />
-    <xacro:include filename="$(find igvc_test_description)/urdf/parts/zed_camera_2i.urdf.xacro" />
+    <!-- <xacro:include filename="$(find igvc_test_description)/urdf/parts/zed_camera_2i.urdf.xacro" /> -->
     <xacro:arg name="hardware_interface" default="IsaacDriveHardware" />
     <xacro:robot_body />

Commit message: name

File: src/igvc_test_description/urdf/parts/zed_camera_x.urdf.xacro (robot description, xacro)
@@ -6,7 +6,7 @@
             <gnss_origin xyz="0 0 0" rpy="0 0 0"/>
         </xacro:zed_camera>
-        <joint name="${prefix}_zed_camera_x_joint" type="fixed">
+        <joint name="${prefix}_zed_camera_2i_joint" type="fixed">
             <parent link="${parent}"/>
-            <child link="${prefix}_zed_camera_x_camera_link"/>
+            <child link="${prefix}_zed_camera_2i_camera_link"/>
             <xacro:insert_block name="origin"/>
         </joint>
