Commit message: added chassis link

File: src/igvc_test_description/urdf/parts/test_robot_body.urdf.xacro (robot description, xacro)
@@ -4,5 +4,5 @@
   <joint name="caster_raceway_joint" type="continuous">
     <origin xyz="0.0011449 -0.3728886 -0.0307033" rpy="0. 0. 0."/>
-    <parent link="temp"/>
+    <parent link="chassis_link"/>
     <child link="caster_raceway_link"/>
     <axis xyz="0. 0. 1."/>
@@ -16,5 +16,5 @@
   <joint name="left_wheel_joint" type="continuous">
     <origin xyz="0.2844359 0.1500906 -0.1274171" rpy="0. 0. 0."/>
-    <parent link="temp"/>
+    <parent link="chassis_link"/>
     <child link="left_wheel_link"/>
     <axis xyz="1. 0. 0."/>
@@ -22,5 +22,5 @@
   <joint name="right_wheel_joint" type="continuous">
     <origin xyz="-0.2918941 0.1492591 -0.1296445" rpy="0. 0. 0."/>
-    <parent link="temp"/>
+    <parent link="chassis_link"/>
     <child link="right_wheel_link"/>
     <axis xyz="1. 0. 0."/>
@@ -28,5 +28,5 @@
   <joint name="rootJoint" type="fixed">
     <origin xyz="0. 0. 0." rpy="0. 0. -0."/>
-    <parent link="temp"/>
+    <parent link="chassis_link"/>
     <child link="base_link"/>
   </joint>
@@ -108,5 +108,5 @@
     </collision>
   </link>
-  <link name="temp">
+  <link name="chassis_link">
     <inertial>
       <origin xyz="0. 0. 0." rpy="0. 0. 0."/>

Commit message: fixed base link

File: src/igvc_test_description/urdf/parts/test_robot_body.urdf.xacro (robot description, xacro)
@@ -28,6 +28,6 @@
   <joint name="rootJoint" type="fixed">
     <origin xyz="0. 0. 0." rpy="0. 0. -0."/>
-    <parent link="chassis_link"/>
-    <child link="base_link"/>
+    <parent link="base_link"/>
+    <child link="chassis_link"/>
   </joint>
   <link name="base_link"/>

Commit message: clean up

File: src/igvc_test_description/urdf/parts/test_robot_body.urdf.xacro (robot description, xacro)
@@ -1,130 +1,130 @@
-<?xml version="1.0" encoding="UTF-8"?>
+<?xml version='1.0' encoding='utf-8'?>
 <robot xmlns:xacro="http://www.ros.org/wiki/xacro">
-    <xacro:macro name="robot_body">
-  <joint name="caster_raceway_joint" type="continuous">
-    <origin xyz="0.0011449 -0.3728886 -0.0307033" rpy="0. 0. 0."/>
-    <parent link="chassis_link"/>
-    <child link="caster_raceway_link"/>
-    <axis xyz="0. 0. 1."/>
-  </joint>
-  <joint name="caster_wheel_joint" type="continuous">
-    <origin xyz="-0.0452015 0.004609 -0.1223279" rpy="-1.5707961 -0.0862496 2.4779847"/>
-    <parent link="caster_raceway_link"/>
-    <child link="caster_wheel_link"/>
-    <axis xyz="0. 0. 1."/>
-  </joint>
-  <joint name="left_wheel_joint" type="continuous">
-    <origin xyz="0.2844359 0.1500906 -0.1274171" rpy="0. 0. 0."/>
-    <parent link="chassis_link"/>
-    <child link="left_wheel_link"/>
-    <axis xyz="1. 0. 0."/>
-  </joint>
-  <joint name="right_wheel_joint" type="continuous">
-    <origin xyz="-0.2918941 0.1492591 -0.1296445" rpy="0. 0. 0."/>
-    <parent link="chassis_link"/>
-    <child link="right_wheel_link"/>
-    <axis xyz="1. 0. 0."/>
-  </joint>
-  <joint name="rootJoint" type="fixed">
-    <origin xyz="0. 0. 0." rpy="0. 0. -0."/>
-    <parent link="base_link"/>
-    <child link="chassis_link"/>
-  </joint>
-  <link name="base_link"/>
-  <link name="caster_raceway_link">
-    <inertial>
-      <origin xyz="-0.0118137 0.0087306 -0.0584325" rpy="0. 0. 0."/>
-      <mass value="0.2597675"/>
-      <inertia ixx="0.0003673" ixy="0.0001647" ixz="0." iyy="0.0004492" iyz="-0." izz="0.0006678"/>
-    </inertial>
-    <visual>
-      <origin xyz="-0.0011449 0.0003886 -0.0088217" rpy="0. 0. -0.663608"/>
-      <geometry>
-        <mesh filename="package://igvc_test_description/meshes/caster_raceway_link_Part_2_Part_2.obj" scale="1. 1. 1."/>
-      </geometry>
-    </visual>
-    <collision>
-      <origin xyz="-0.0011449 0.0003886 -0.0088217" rpy="0. 0. -0.663608"/>
-      <geometry>
-        <mesh filename="package://igvc_test_description/meshes/caster_raceway_link_Part_2_Part_2.obj" scale="1. 1. 1."/>
-      </geometry>
-    </collision>
-  </link>
-  <link name="caster_wheel_link">
-    <inertial>
-      <origin xyz="-0. -0. -0.0238125" rpy="0. 0. 0."/>
-      <mass value="1.0005643"/>
-      <inertia ixx="0.0017247" ixy="-0." ixz="0." iyy="0.0030953" iyz="-0." izz="0.0017247"/>
-    </inertial>
-    <visual>
-      <origin xyz="0.0373062 0.1135063 -0.0238125" rpy="-1.5707965 -0.0000001 0. "/>
-      <geometry>
-        <mesh filename="package://igvc_test_description/meshes/caster_wheel_link__in_Caster__in_Caster.obj" scale="1. 1. 1."/>
-      </geometry>
-    </visual>
-    <collision>
-      <origin xyz="0.0373062 0.1135063 -0.0238125" rpy="-1.5707965 -0.0000001 0. "/>
-      <geometry>
-        <mesh filename="package://igvc_test_description/meshes/caster_wheel_link__in_Caster__in_Caster.obj" scale="1. 1. 1."/>
-      </geometry>
-    </collision>
-  </link>
-  <link name="left_wheel_link">
-    <inertial>
-      <origin xyz="-0.0010859 -0.0000906 -0.0010079" rpy="0. 0. 0."/>
-      <mass value="2.1118586"/>
-      <inertia ixx="0.0059185" ixy="-0." ixz="-0." iyy="0.0086441" iyz="0.0022525" izz="0.00778"/>
-    </inertial>
-    <visual>
-      <origin xyz="-0.0010859 -0.0000906 -0.0010079" rpy="0. 0.8801533 1.5707964"/>
-      <geometry>
-        <mesh filename="package://igvc_test_description/meshes/left_wheel_link__in_Wheel_Stand_In_01__in_Wheel_Stand_In.obj" scale="1. 1. 1."/>
-      </geometry>
-    </visual>
-    <collision>
-      <origin xyz="-0.0010859 -0.0000906 -0.0010079" rpy="0. 0.8801533 1.5707964"/>
-      <geometry>
-        <mesh filename="package://igvc_test_description/meshes/left_wheel_link__in_Wheel_Stand_In_01__in_Wheel_Stand_In.obj" scale="1. 1. 1."/>
-      </geometry>
-    </collision>
-  </link>
-  <link name="right_wheel_link">
-    <inertial>
-      <origin xyz="0.0085441 0.0007409 0.0012195" rpy="0. 0. 0."/>
-      <mass value="2.1118586"/>
-      <inertia ixx="0.0059185" ixy="-0." ixz="0." iyy="0.0059185" iyz="-0." izz="0.0105056"/>
-    </inertial>
-    <visual>
-      <origin xyz="0.0085441 0.0007409 0.0012195" rpy="3.1415927 0. -1.5707964"/>
-      <geometry>
-        <mesh filename="package://igvc_test_description/meshes/right_wheel_link__in_Wheel_Stand_In_01__in_Wheel_Stand_In.obj" scale="1. 1. 1."/>
-      </geometry>
-    </visual>
-    <collision>
-      <origin xyz="0.0085441 0.0007409 0.0012195" rpy="3.1415927 0. -1.5707964"/>
-      <geometry>
-        <mesh filename="package://igvc_test_description/meshes/right_wheel_link__in_Wheel_Stand_In_01__in_Wheel_Stand_In.obj" scale="1. 1. 1."/>
-      </geometry>
-    </collision>
-  </link>
-  <link name="chassis_link">
-    <inertial>
-      <origin xyz="0. 0. 0." rpy="0. 0. 0."/>
-      <mass value="20."/>
-      <inertia ixx="0.001" ixy="0." ixz="0." iyy="0.001" iyz="0." izz="0.001"/>
-    </inertial>
-    <visual>
-      <origin xyz="0. 0. 0." rpy="0. 0. 0."/>
-      <geometry>
-        <mesh filename="package://igvc_test_description/meshes/_FE2CBA3_2B86_49A6_86C6_46C335366A6A.obj" scale="1. 1. 1."/>
-      </geometry>
-    </visual>
-    <collision>
-      <origin xyz="0. 0. 0." rpy="0. 0. 0."/>
-      <geometry>
-        <mesh filename="package://igvc_test_description/meshes/_FE2CBA3_2B86_49A6_86C6_46C335366A6A.obj" scale="1. 1. 1."/>
-      </geometry>
-    </collision>
-  </link>
-    </xacro:macro>
+  <xacro:macro name="robot_body">
+    <joint name="caster_raceway_joint" type="continuous">
+      <origin xyz="0.3728886 0.0011449 -0.0307033" rpy="0. 0. 0." />
+      <parent link="chassis_link" />
+      <child link="caster_raceway_link" />
+      <axis xyz="0. 0. 1" />
+    </joint>
+    <joint name="caster_wheel_joint" type="continuous">
+      <origin xyz="-0.03 -0.0252015 -0.1223279" rpy="1.570794 -1.570794 0" />
+      <parent link="caster_raceway_link" />
+      <child link="caster_wheel_link" />
+      <axis xyz="0. 0. 1" />
+    </joint>
+    <joint name="left_wheel_joint" type="continuous">
+      <origin xyz="-0.1500906 0.2844359 -0.1274171" rpy="0. 0. 0." />
+      <parent link="chassis_link" />
+      <child link="left_wheel_link" />
+      <axis xyz="0. 1 0." />
+    </joint>
+    <joint name="right_wheel_joint" type="continuous">
+      <origin xyz="-0.1492591 -0.2918941 -0.1296445" rpy="0. 0. 0." />
+      <parent link="chassis_link" />
+      <child link="right_wheel_link" />
+      <axis xyz="0. 1 0." />
+    </joint>
+    <joint name="rootJoint" type="fixed">
+      <origin xyz="0. 0. 0." rpy="0. 0. 0." />
+      <parent link="base_link" />
+      <child link="chassis_link" />
+    </joint>
+    <link name="base_link" />
+    <link name="caster_raceway_link">
+      <inertial>
+        <origin xyz="-0.0087306 -0.0118137 -0.0584325" rpy="0. 0. 1.570796" />
+        <mass value="0.2597675" />
+        <inertia ixx="0.0003673" ixy="0.0001647" ixz="0." iyy="0.0004492" iyz="-0." izz="0.0006678" />
+      </inertial>
+      <visual>
+        <origin xyz="-0.0003886 -0.0011449 -0.0088217" rpy="0. 0. ${0.9071883-3.14152/4}" />
+        <geometry>
+          <mesh filename="file:///home/nitin-5090/Documents/DevEnv/jazzy_ws/IGVC_robot_2026/src/igvc_test_description/meshes/caster_raceway_link_Part_2_Part_2.obj" scale="1. 1. 1." />
+        </geometry>
+      </visual>
+      <collision>
+        <origin xyz="-0.0003886 -0.0011449 -0.0088217" rpy="0. 0. ${0.9071883-3.14152/4}" />
+        <geometry>
+          <mesh filename="file:///home/nitin-5090/Documents/DevEnv/jazzy_ws/IGVC_robot_2026/src/igvc_test_description/meshes/caster_raceway_link_Part_2_Part_2.obj" scale="1. 1. 1." />
+        </geometry>
+      </collision>
+    </link>
+    <link name="caster_wheel_link">
+      <inertial>
+        <origin xyz="0. 0. -0.0238125" rpy="0. 0. 1.570796" />
+        <mass value="1.0005643" />
+        <inertia ixx="0.0017247" ixy="-0." ixz="0." iyy="0.0030953" iyz="-0." izz="0.0017247" />
+      </inertial>
+      <visual>
+        <origin xyz="-0.1135063 0.0373062 -0.0238125" rpy="-1.570796 -1e-07 1.570796" />
+        <geometry>
+          <mesh filename="file:///home/nitin-5090/Documents/DevEnv/jazzy_ws/IGVC_robot_2026/src/igvc_test_description/meshes/caster_wheel_link__in_Caster__in_Caster.obj" scale="1. 1. 1." />
+        </geometry>
+      </visual>
+      <collision>
+        <origin xyz="-0.1135063 0.0373062 -0.0238125" rpy="-1.570796 -1e-07 1.570796" />
+        <geometry>
+          <mesh filename="file:///home/nitin-5090/Documents/DevEnv/jazzy_ws/IGVC_robot_2026/src/igvc_test_description/meshes/caster_wheel_link__in_Caster__in_Caster.obj" scale="1. 1. 1." />
+        </geometry>
+      </collision>
+    </link>
+    <link name="left_wheel_link">
+      <inertial>
+        <origin xyz="9.06e-05 -0.0010859 -0.0010079" rpy="0. 0. 1.570796" />
+        <mass value="2.1118586" />
+        <inertia ixx="0.0059185" ixy="-0." ixz="-0." iyy="0.0086441" iyz="0.0022525" izz="0.00778" />
+      </inertial>
+      <visual>
+        <origin xyz="9.06e-05 -0.0010859 -0.0010079" rpy="0. 0.8801533 -3.141593" />
+        <geometry>
+          <mesh filename="file:///home/nitin-5090/Documents/DevEnv/jazzy_ws/IGVC_robot_2026/src/igvc_test_description/meshes/left_wheel_link__in_Wheel_Stand_In_01__in_Wheel_Stand_In.obj" scale="1. 1. 1." />
+        </geometry>
+      </visual>
+      <collision>
+        <origin xyz="9.06e-05 -0.0010859 -0.0010079" rpy="0. 0.8801533 -3.141593" />
+        <geometry>
+          <mesh filename="file:///home/nitin-5090/Documents/DevEnv/jazzy_ws/IGVC_robot_2026/src/igvc_test_description/meshes/left_wheel_link__in_Wheel_Stand_In_01__in_Wheel_Stand_In.obj" scale="1. 1. 1." />
+        </geometry>
+      </collision>
+    </link>
+    <link name="right_wheel_link">
+      <inertial>
+        <origin xyz="-0.0007409 0.0085441 0.0012195" rpy="0. 0. 1.570796" />
+        <mass value="2.1118586" />
+        <inertia ixx="0.0059185" ixy="-0." ixz="0." iyy="0.0059185" iyz="-0." izz="0.0105056" />
+      </inertial>
+      <visual>
+        <origin xyz="-0.0007409 0.0085441 0.0012195" rpy="-3.141593 0. -7.32051e-08" />
+        <geometry>
+          <mesh filename="file:///home/nitin-5090/Documents/DevEnv/jazzy_ws/IGVC_robot_2026/src/igvc_test_description/meshes/right_wheel_link__in_Wheel_Stand_In_01__in_Wheel_Stand_In.obj" scale="1. 1. 1." />
+        </geometry>
+      </visual>
+      <collision>
+        <origin xyz="-0.0007409 0.0085441 0.0012195" rpy="-3.141593 0. -7.32051e-08" />
+        <geometry>
+          <mesh filename="file:///home/nitin-5090/Documents/DevEnv/jazzy_ws/IGVC_robot_2026/src/igvc_test_description/meshes/right_wheel_link__in_Wheel_Stand_In_01__in_Wheel_Stand_In.obj" scale="1. 1. 1." />
+        </geometry>
+      </collision>
+    </link>
+    <link name="chassis_link">
+      <inertial>
+        <origin xyz="0. 0. 0." rpy="0. 0. 1.570796" />
+        <mass value="20." />
+        <inertia ixx="0.001" ixy="0." ixz="0." iyy="0.001" iyz="0." izz="0.001" />
+      </inertial>
+      <visual>
+        <origin xyz="0. 0. 0." rpy="0. 0. 1.570796" />
+        <geometry>
+          <mesh filename="file:///home/nitin-5090/Documents/DevEnv/jazzy_ws/IGVC_robot_2026/src/igvc_test_description/meshes/_FE2CBA3_2B86_49A6_86C6_46C335366A6A.obj" scale="1. 1. 1." />
+        </geometry>
+      </visual>
+      <collision>
+        <origin xyz="0. 0. 0." rpy="0. 0. 1.570796" />
+        <geometry>
+          <mesh filename="file:///home/nitin-5090/Documents/DevEnv/jazzy_ws/IGVC_robot_2026/src/igvc_test_description/meshes/_FE2CBA3_2B86_49A6_86C6_46C335366A6A.obj" scale="1. 1. 1." />
+        </geometry>
+      </collision>
+    </link>
+  </xacro:macro>
 </robot>

File: src/igvc_test_description/urdf/robots/test_robot.urdf.xacro (robot description, xacro)
@@ -7,11 +7,11 @@
     <xacro:robot_body />
     <xacro:zed_camera_x parent="chassis_link" prefix="left">
-        <origin xyz="0.2 -0.1 ${3.14/2}" rpy="0 0 0"/>
+        <origin xyz="0.4 0.16 0.034" rpy="0 0 ${3.14*13/36}"/>
     </xacro:zed_camera_x>
     <xacro:zed_camera_x parent="chassis_link" prefix="front">
-        <origin xyz="0.2 0 0" rpy="0 0 0"/>
+        <origin xyz="0.47 0 0.034" rpy="0 0 0"/>
     </xacro:zed_camera_x>
     <xacro:zed_camera_x parent="chassis_link" prefix="right">
-        <origin xyz="0.2 0.1 -${3.14/2}" rpy="0 0 0"/>
+        <origin xyz="0.4 -0.16 0.034" rpy="0 0 -${3.14*13/36}"/>
     </xacro:zed_camera_x>
 </robot>

Commit message: added new sensors need to tune values slightly

File: src/igvc_test_description/urdf/parts/test_robot_body.urdf.xacro (robot description, xacro)
@@ -120,4 +120,22 @@
         </geometry>
       </visual>
+      <visual>
+        <origin xyz="0.13 0. 0.005" rpy="0. 0. 0." />
+        <geometry>
+          <box size="0.9 0.45 0.01" />
+        </geometry>
+      </visual>
+      <visual>
+        <origin xyz="0.225 0. 0.085" rpy="0. 0. 0." />
+        <geometry>
+          <box size="0.45 0.45 0.15" />
+        </geometry>
+      </visual>
+      <visual>
+        <origin xyz="0.225 0. 0.31" rpy="0. 0. 0." />
+        <geometry>
+          <box size="0.05 0.05 0.3" />
+        </geometry>
+      </visual>
       <collision>
         <origin xyz="0. 0. 0." rpy="0. 0. 1.570796" />

File: src/igvc_test_description/urdf/robots/test_robot.urdf.xacro (robot description, xacro)
@@ -4,14 +4,22 @@
     <xacro:include filename="$(find igvc_test_description)/urdf/control/ros2_control_info.urdf.xacro" />
     <xacro:include filename="$(find igvc_test_description)/urdf/parts/zed_camera_x.urdf.xacro" />
+    <xacro:include filename="$(find igvc_test_description)/urdf/parts/rplidar_c1.urdf.xacro" />
+    <xacro:include filename="$(find igvc_test_description)/urdf/parts/gps_antenna.urdf.xacro" />
     <xacro:arg name="hardware_interface" default="IsaacDriveHardware" />
     <xacro:robot_body />
     <xacro:zed_camera_x parent="chassis_link" prefix="left">
-        <origin xyz="0.4 0.16 0.034" rpy="0 0 ${3.14*13/36}"/>
+        <origin xyz="0.4 0.2 0.194" rpy="0 ${3.14/18} ${3.14*95/180}"/>
     </xacro:zed_camera_x>
     <xacro:zed_camera_x parent="chassis_link" prefix="front">
-        <origin xyz="0.47 0 0.034" rpy="0 0 0"/>
+        <origin xyz="0.45 0 0.194" rpy="0 0 0"/>
     </xacro:zed_camera_x>
     <xacro:zed_camera_x parent="chassis_link" prefix="right">
-        <origin xyz="0.4 -0.16 0.034" rpy="0 0 -${3.14*13/36}"/>
+        <origin xyz="0.4 -0.2 0.194" rpy="0 ${3.14/18} -${3.14*95/180}"/>
     </xacro:zed_camera_x>
+    <xacro:rplidar_c1 parent="chassis_link" prefix="top">
+        <origin xyz="0.225 0 0.46" rpy="0 0 0"/>
+    </xacro:rplidar_c1>
+    <xacro:gps_antenna parent="chassis_link" prefix="front">
+        <origin xyz="0.2 -0.15 0.16" rpy="0 0 0"/>
+    </xacro:gps_antenna>
 </robot>

Commit message: final changes

File: src/igvc_test_description/urdf/parts/test_robot_body.urdf.xacro (robot description, xacro)
@@ -133,7 +133,7 @@
       </visual>
       <visual>
-        <origin xyz="0.225 0. 0.31" rpy="0. 0. 0." />
+        <origin xyz="0.34 0. 0.52" rpy="0. 0. 0." />
         <geometry>
-          <box size="0.05 0.05 0.3" />
+          <box size="0.05 0.05 0.5" />
         </geometry>
       </visual>

File: src/igvc_test_description/urdf/robots/test_robot.urdf.xacro (robot description, xacro)
@@ -22,5 +22,5 @@
     </xacro:zed_camera_2i>
     <xacro:rplidar_c1 parent="chassis_link" prefix="top">
-        <origin xyz="0.225 0 0.46" rpy="0 0 0"/>
+        <origin xyz="0.345 0 0.52" rpy="0 0 0"/>
     </xacro:rplidar_c1>
     <xacro:gps_antenna parent="chassis_link" prefix="front">
